File: STM32WB-Bluetooth_Hardware_Design_pcb/STM32WB-Bluetooth_Hardware_Design.kicad_pcb (KiCad board)
At the start: 2 copper layers, 0 parts

Commit message: Final schematics and the pcb
Parts:
- added C1: 4u7, Capacitor_SMD:C_0603_1608Metric, F.Cu at (49.6, 71.2)
- added C10: 4u7, Capacitor_SMD:C_0603_1608Metric, F.Cu at (66.2, 62.5)
- added C11: 100n, Capacitor_SMD:C_0402_1005Metric, F.Cu at (67.3, 65.0)
- added C12: 100n, Capacitor_SMD:C_0402_1005Metric, F.Cu at (75.2, 67.5)
- added C13: 10p, Capacitor_SMD:C_0402_1005Metric, F.Cu at (68.8, 75.2)
- added C14: 10p, Capacitor_SMD:C_0402_1005Metric, F.Cu at (66.3, 75.2)
- added C15: 100n, Capacitor_SMD:C_0402_1005Metric, F.Cu at (63.8, 77.7)
- added C16: 4u7, Capacitor_SMD:C_0603_1608Metric, F.Cu at (70.8, 64.5)
- added C17: 0.8p, Capacitor_SMD:C_0402_1005Metric, F.Cu at (76.5, 69.2)
- added C18: 0.3p, Capacitor_SMD:C_0402_1005Metric, F.Cu at (79.5, 69.2)
- added C19: 100n, Capacitor_SMD:C_0402_1005Metric, F.Cu at (64.0, 80.5)
- added C2: 4u7, Capacitor_SMD:C_0603_1608Metric, F.Cu at (52.2, 74.3)
- added C3: 4u7, Capacitor_SMD:C_0603_1608Metric, F.Cu at (63.8, 75.2)
- added C4: 100n, Capacitor_SMD:C_0402_1005Metric, F.Cu at (64.0, 68.8)
- added C5: 100n, Capacitor_SMD:C_0402_1005Metric, F.Cu at (71.7, 75.3)
- added C6: 100n, Capacitor_SMD:C_0402_1005Metric, F.Cu at (63.8, 72.8)
- added C7: 100n, Capacitor_SMD:C_0402_1005Metric, F.Cu at (67.3, 64.0)
- added C8: 100n, Capacitor_SMD:C_0402_1005Metric, F.Cu at (65.0, 72.8)
- added C9: 100n, Capacitor_SMD:C_0402_1005Metric, F.Cu at (74.9, 70.0)
- added D1: LED, LED_SMD:LED_0402_1005Metric, F.Cu at (79.2, 75.8)
- added FLT1: DLF162500LT-5028A1, STM32WB-Bluetooth_Hardware_Design_SchematicFootprints:DLF162500LT-5028A1, F.Cu at (81.3, 68.8)
- added FM1: Fiducial, Fiducial:Fiducial_0.5mm_Mask1mm, F.Cu at (44.2, 61.5)
- added FM2: Fiducial, Fiducial:Fiducial_0.5mm_Mask1mm, F.Cu at (80.0, 61.5)
- added FM3: Fiducial, Fiducial:Fiducial_0.5mm_Mask1mm, F.Cu at (80.0, 82.2)
- added G***: LOGO, Assets:Ucaselabs_8mm_2mm, F.Cu at (58.7, 79.5)
- added G***: LOGO, Assets:UA_Fill_2mm_2mm, F.Cu at (72.8, 82.5)
- added H1: MountingHole_Pad, MountingHole:MountingHole_2.2mm_M2_Pad_Via, F.Cu at (51.0, 63.2)
- added H2: MountingHole_Pad, MountingHole:MountingHole_2.2mm_M2_Pad_Via, F.Cu at (51.0, 81.8)
- added H3: MountingHole_Pad, MountingHole:MountingHole_2.2mm_M2_Pad_Via, F.Cu at (84.2, 81.8)
- added H4: MountingHole_Pad, MountingHole:MountingHole_2.2mm_M2_Pad_Via, F.Cu at (84.2, 63.0)
- added J1: USB_C_Receptacle_USB2.0_16P, Connector_USB:USB_C_Receptacle_GCT_USB4105-xx-A_16P_TopMnt_Horizontal, F.Cu at (40.7, 68.0)
- added J2: Conn_ARM_SWD_TagConnect_TC2030, Connector:Tag-Connect_TC2030-IDC-FP_2x03_P1.27mm_Vertical, F.Cu at (58.7, 70.0)
- added J3: Conn_01x04, Connector_Molex:Molex_PicoBlade_53048-0410_1x04_P1.25mm_Horizontal, F.Cu at (44.0, 78.1)
- added J4: Conn_Coaxial, Connector_Coaxial:U.FL_Hirose_U.FL-R-SMT-1_Vertical, F.Cu at (84.5, 68.8)
- added L1: 10n, Inductor_SMD:L_0402_1005Metric, F.Cu at (68.8, 64.5)
- added L2: 10u, Inductor_SMD:L_0805_2012Metric, F.Cu at (69.8, 62.5)
- added L3: 2.7n, Inductor_SMD:L_0402_1005Metric, F.Cu at (78.0, 68.8)
- added R1: 5.1k, Resistor_SMD:R_0402_1005Metric, F.Cu at (41.7, 74.2)
- added R2: 5.1k, Resistor_SMD:R_0402_1005Metric, F.Cu at (41.6, 61.8)
- added R3: 220R, Resistor_SMD:R_0402_1005Metric, F.Cu at (80.5, 75.8)
- added R4: 220R, Resistor_SMD:R_0402_1005Metric, F.Cu at (73.5, 75.8)
- added R5: 220R, Resistor_SMD:R_0402_1005Metric, F.Cu at (74.7, 75.8)
- added R6: 5.1k, Resistor_SMD:R_0402_1005Metric, F.Cu at (63.2, 82.5)
- added R7: 220R, Resistor_SMD:R_0402_1005Metric, F.Cu at (64.8, 82.5)
- added SW1: SW_Push, Button_Switch_SMD:SW_SPST_B3U-1000P, F.Cu at (68.5, 82.0)
- added U1: USBLC6-2SC6, Package_TO_SOT_SMD:SOT-23-6, F.Cu at (49.4, 68.0)
- added U2: MIC5365-3.3YD5, Package_TO_SOT_SMD:SOT-23-5, F.Cu at (49.5, 74.2)
- added U3: STM32WB55CEU6, Package_DFN_QFN:QFN-48-1EP_7x7mm_P0.5mm_EP5.6x5.6mm, F.Cu at (70.0, 70.0)
- added X1: 32KHz768, Crystal:Crystal_SMD_2012-2Pin_2.0x1.2mm, F.Cu at (67.5, 76.8)
- added X2: 32MHz, Crystal:Crystal_SMD_2016-4Pin_2.0x1.6mm, F.Cu at (75.0, 63.8)
- added kibuzzard-663E8D7A: G***, kibuzzard-663E8D7A, F.Cu at (58.5, 64.9)
- added kibuzzard-663E8D97: G***, kibuzzard-663E8D97, F.Cu at (47.2, 79.6)
- added kibuzzard-663E8DAE: G***, kibuzzard-663E8DAE, F.Cu at (47.3, 65.0)
- added kibuzzard-663E8DF2: G***, kibuzzard-663E8DF2, F.Cu at (69.3, 79.2)
- added kibuzzard-663E8E0C: G***, kibuzzard-663E8E0C, F.Cu at (85.9, 73.3)
Routing:
- net /UART_RXC: track 0.00 -> 34.1 mm
- net /UART_TXC: track 0.00 -> 32.8 mm
- net /SWD_NRST: track 0.00 -> 31.2 mm
- net GND: track 0.00 -> 28.0 mm, vias 0 -> 115
- net +3V3: track 0.00 -> 25.5 mm, vias 0 -> 12
- net +5V: track 0.00 -> 21.9 mm
- net /USB_D-: track 0.00 -> 19.4 mm
- net /USB_D+: track 0.00 -> 19.4 mm
- net /BOOT0: track 0.00 -> 15.8 mm, vias 0 -> 2
- net /SWD_TRC: track 0.00 -> 11.3 mm
- net /SWD_DIO: track 0.00 -> 10.7 mm
- net /SWD_CLK: track 0.00 -> 8.59 mm
- net /LED_A: track 0.00 -> 8.33 mm
- net /USB_CC1: track 0.00 -> 6.89 mm
- net /USBC_D-: track 0.00 -> 6.67 mm
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- added copper zone on B.Cu, net +3V3
- added copper zone on F.Cu, net +3V3
- added copper zone on F.Cu, net /SMPSFB
- added copper zone on F.Cu, net GND
- added copper zone on In1.Cu, net GND
- added copper zone on In2.Cu, net GND
Other:
- board outline added: 50 x 25 mm
- copper layers 2 -> 4
- rule pad_to_mask_clearance: 0 -> 0.08
- board text added: "2024/05/11"
- board text added: "Designed By:"
- board text added: "Rev.1.0"
