File: STM32WB-Bluetooth_Hardware_Design_pcb/STM32WB-Bluetooth_Hardware_Design.kicad_sch (KiCad schematic)
At the start: 11 parts, among them U1 STM32WB55CEU6

Commit message: Final schematics and the pcb
Parts:
- added C1, C16, C2: 4u7, Capacitor_SMD:C_0603_1608Metric, symbol Device:C
- added C13, C14: 10p, Capacitor_SMD:C_0402_1005Metric, symbol Device:C
- added C15, C19: 100n, Capacitor_SMD:C_0402_1005Metric, symbol Device:C
- added C17: 0.8p, Capacitor_SMD:C_0402_1005Metric, symbol Device:C
- added C18: 0.3p, Capacitor_SMD:C_0402_1005Metric, symbol Device:C
- added D1: LED, LED_SMD:LED_0402_1005Metric, symbol Device:LED
- added FLT1: DLF162500LT-5028A1, STM32WB-Bluetooth_Hardware_Design_SchematicFootprints:DLF162500LT-5028A1, symbol STM32WB-Bluetooth_Hardware_Design_SchematicSymbols:DLF162500LT-5028A1
- added FM1, FM2, FM3: Fiducial, Fiducial:Fiducial_0.5mm_Mask1mm, symbol Mechanical:Fiducial
- added H1, H2, H3, H4: MountingHole_Pad, MountingHole:MountingHole_2.2mm_M2_Pad_Via, symbol Mechanical:MountingHole_Pad
- added J1: USB_C_Receptacle_USB2.0_16P, Connector_USB:USB_C_Receptacle_GCT_USB4105-xx-A_16P_TopMnt_Horizontal, symbol Connector:USB_C_Receptacle_USB2.0_16P
- added J2: Conn_ARM_SWD_TagConnect_TC2030, Connector:Tag-Connect_TC2030-IDC-FP_2x03_P1.27mm_Vertical, symbol Connector:Conn_ARM_SWD_TagConnect_TC2030
- added J3: Conn_01x04, Connector_Molex:Molex_PicoBlade_53048-0410_1x04_P1.25mm_Horizontal, symbol Connector_Generic:Conn_01x04
- added J4: Conn_Coaxial, Connector_Coaxial:U.FL_Hirose_U.FL-R-SMT-1_Vertical, symbol Connector:Conn_Coaxial
- added L1: 10n, Inductor_SMD:L_0402_1005Metric, symbol Device:L
- added L2: 10u, Inductor_SMD:L_0805_2012Metric, symbol Device:L
- added L3: 2.7n, Inductor_SMD:L_0402_1005Metric, symbol Device:L
- added R1, R2, R6: 5.1k, Resistor_SMD:R_0402_1005Metric, symbol Device:R
- added R3, R4, R5, R7: 220R, Resistor_SMD:R_0402_1005Metric, symbol Device:R
- added SW1: SW_Push, Button_Switch_SMD:SW_SPST_B3U-1000P, symbol Switch:SW_Push
- added U1: USBLC6-2SC6, Package_TO_SOT_SMD:SOT-23-6, symbol Power_Protection:USBLC6-2SC6
- added U2: MIC5365-3.3YD5, Package_TO_SOT_SMD:SOT-23-5, symbol Regulator_Linear:MIC5365-3.3YD5
- added X1: 32KHz768, Crystal:Crystal_SMD_2012-2Pin_2.0x1.2mm, symbol Device:Crystal
- added X2: 32MHz, Crystal:Crystal_SMD_2016-4Pin_2.0x1.6mm, symbol Device:Crystal_GND24
- C10: renamed from C8; footprint (none) -> Capacitor_SMD:C_0603_1608Metric
- C11: renamed from C9; footprint (none) -> Capacitor_SMD:C_0402_1005Metric
- C12: renamed from C10; footprint (none) -> Capacitor_SMD:C_0402_1005Metric
- C3: renamed from C7; footprint (none) -> Capacitor_SMD:C_0603_1608Metric
- C4: renamed from C1; footprint (none) -> Capacitor_SMD:C_0402_1005Metric
- C5: renamed from C2; footprint (none) -> Capacitor_SMD:C_0402_1005Metric
- C6: renamed from C3; footprint (none) -> Capacitor_SMD:C_0402_1005Metric
- C7: renamed from C4; footprint (none) -> Capacitor_SMD:C_0402_1005Metric
- C8: renamed from C5; footprint (none) -> Capacitor_SMD:C_0402_1005Metric
- C9: renamed from C6; footprint (none) -> Capacitor_SMD:C_0402_1005Metric
- renumbered U1 to U3
Connections:
- net +3V3: now also C2.1, J2.1 (VCC), J3.1 (Pin_1), SW1.2, U2.5 (VOUT)
- net GND: now also C1.2, C13.2, C14.2, C15.2, C16.2, C17.2, C18.2, C19.2, C2.2, FLT1.2 (GND), FLT1.4 (GND), H1.1, H2.1, H3.1, H4.1, J1.A1 (GND), J1.A12 (GND), J1.B1 (GND), J1.B12 (GND), J1.S1 (SHIELD), J2.5 (GND), J3.4 (Pin_4), J4.2 (Ext), R1.2, R2.2, R3.2, R6.2, U1.2 (GND), U2.2 (GND), X2.2, X2.4
- net UART_TX: now reaches U3.11 (PA2)
- net UART_TX: now also R4.1
- net UART_RX: now reaches U3.12 (PA3)
- net UART_RX: now also R5.1
- net LED_A: now reaches U3.16 (PA7)
- net LED_A: now also D1.2 (A)
- net LSE_IN: now reaches U3.2 (PC14)
- net LSE_IN: now also C14.1, X1.2
- net RF: now reaches U3.21 (RF1)
- net RF: now also C17.1, L3.1
- net HSE_OUT: now reaches U3.24 (OSC_OUT)
- net HSE_OUT: now also X2.1
- net HSE_IN: now reaches U3.25 (OSC_IN)
- net HSE_IN: now also X2.3
- net LSE_OUT: now reaches U3.3 (PC15)
- net LSE_OUT: now also C13.1, X1.1
- net SMPSFB: now reaches U3.31 (VFBSMPS)
- net SMPSFB: now also C16.1, L2.2
- net SMPSLX: now reaches U3.33 (VLXSMPS)
- net SMPSLX: now also L1.1
- net USB_D-: now reaches U3.37 (PA11)
- net USB_D-: now also U1.6 (I/O1)
- net USB_D+: now reaches U3.38 (PA12)
- net USB_D+: now also U1.4 (I/O2)
- net SWD_DIO: now reaches U3.39 (PA13)
- net SWD_DIO: now also J2.2 (SWDIO)
- net BOOT0: now reaches U3.4 (PH3)
- net BOOT0: now also C19.1, R6.1, R7.2
- net SWD_CLK: now reaches U3.41 (PA14)
- net SWD_CLK: now also J2.4 (SWCLK)
- net SWD_TRC: now reaches U3.43 (PB3)
- net SWD_TRC: now also J2.6 (SWO)
- net SWD_NRST: now reaches U3.7 (NRST)
- net SWD_NRST: now also C15.1, J2.3 (~{RESET})
- new net: R7.1, SW1.1
- new net +5V: C1.1, J1.A4 (VBUS), J1.A9 (VBUS), J1.B4 (VBUS), J1.B9 (VBUS), U1.5 (VBUS), U2.1 (VIN), U2.3 (EN)
- new net LED_K: D1.1 (K), R3.1
- new net RF_ANT: FLT1.3 (OUT), J4.1 (In)
- new net RF_MATCH: C18.1, FLT1.1 (IN), L3.2
- new net SMPSLXL: L1.2, L2.1
- new net UART_RXC: J3.3 (Pin_3), R5.2
- new net UART_TXC: J3.2 (Pin_2), R4.2
- new net USBC_D+: J1.A6 (D+), J1.B6 (D+), U1.3 (I/O2)
- new net USBC_D-: J1.A7 (D-), J1.B7 (D-), U1.1 (I/O1)
- new net USB_CC1: J1.A5 (CC1), R2.1
- new net USB_CC2: J1.B5 (CC2), R1.1
- no-connect marks 0 -> 21
Other:
- note added: "(3.3-1.8)/220 ~= 7mA"
- note added: "Add a series resistor here though it may be of 0 ohm for the sake of longivity of the crystal."
- note added: "Boot0 Switch"
- note added: "LSE(32.768KHz) & HSE(32MHz) Crystals"
- note added: "Tag-Connect SWD Header"
- note added: "U.fl Connector"
- note added: "UART Header"
- note added: "USB-C Connector"
- company: (none) -> Ucase Labs
- title: (none) -> STM32B KiCad Tutorial
- moved on the sheet: C10, C11, C12, C3, C4, C5, C6, C7, C8, C9, U3
