File: Easyeda_nfc_pcb/Easyeda_nfc_pcb.kicad_pcb (KiCad board)
At the start: 2 copper layers, 86 x 52 mm, 5 parts, among them U1 NT3H2111W0FHKH

Commit message: exported images for better visualization
Parts:
- added G***: LOGO, Assets:ua_linktree_16mm_16mm, F.Cu at (181.0, 118.0)
